File: steeringWheel/steeringWheelPCB/TEST_newWheelBoard.kicad_pcb (KiCad board)
At the start: 2 copper layers, 85 x 58 mm, 38 parts, among them J1 Conn_01x20_Female_OLED, J10 Conn_02x01_Left_Black, J11 Conn_02x01_Blue, J12 Conn_02x01_Green, J13 Conn_02x01_Red, J14 Conn_02x01_Right_Black, J2 Conn_01x09_Female_LED_Right, J3 Conn_01x09_Female_LED_Left, J4 Conn_01x06_Female_Abs_Pos, J5 Conn_02x01_Yellow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

Commit message: Uploading daq KiCad Project
I forgot I generated these files awhile ago (no one from the team bugged me about them, which is a little concerning). Uploading after opening to verify files were complete.
Parts:
- C2: value 10uF -> 22uF
