File: daq/MAIN_daq.kicad_pcb (KiCad board)
At the start: 2 copper layers, 116.2 x 57 mm, 30 parts, among them J1 Conn_01x14_Male, J2 Conn_01x14_Male, J3 Conn_02x20_Odd_Even_RPi, U1 Teensy4.0, U2 LM7805_TO220, U3 MCP2551-I-P

Commit message: Uploaded DAQ KiCad Project
After my initial upload of these files, I realized that some of the files were not like I left them in May 2021 (just some text on the silk screen layers was missing. Couldn't find any backups so re-added the text and replotted gerbers to make sure all files were correct).
Other:
- board text added: "NOTE: For 0 - 3.3V analog inputs, use the solderable jumper (R2, R4, R8, R10). For 0 - 5V analog inputs, do NOT use the solderable jumper."
- board text added: "Tufts Electric Racing - DAQ Main Board v1.0 By: Martin Majkut - Date: Spring 2021"
